File: FRC_I2C_Mux.kicad_sch (KiCad schematic)
At the start: 46 parts, among them J1 Conn_01x04, J10 Conn_01x04, J11 Conn_01x04, J12 Conn_01x02, J2 Conn_01x04, J3 Conn_01x04, J4 Conn_01x04, J5 Conn_01x04, J6 Conn_01x02, J7 Conn_01x02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

Commit message: Fix footprint paths
Parts:
- D1: footprint SamacSys_Parts:LEDC1006X25N -> footprints:LEDC1006X25N
- RN1, RN2: footprint SamacSys_Parts:EXB2HV_1 -> footprints:EXB2HV_1
Changed lines of the file:
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@@
     (property "Reference" "RN1" (id 0) (at 134.62 39.37 90))
     (property "Value" "R_Pack08" (id 1) (at 134.62 41.91 90))
-    (property "Footprint" "SamacSys_Parts:EXB2HV_1" (id 2) (at 134.62 67.945 90)
+    (property "Footprint" "footprints:EXB2HV_1" (id 2) (at 134.62 67.945 90)
       (effects (font (size 1.27 1.27)) hide)
     )
@@
     (property "Reference" "D1" (id 0) (at 136.8425 115.57 0))
     (property "Value" "LED" (id 1) (at 136.8425 118.11 0))
-    (property "Footprint" "SamacSys_Parts:LEDC1006X25N" (id 2) (at 138.43 121.92 0)
+    (property "Footprint" "footprints:LEDC1006X25N" (id 2) (at 138.43 121.92 0)
       (effects (font (size 1.27 1.27)) hide)
     )
@@
     (property "Reference" "RN2" (id 0) (at 134.62 90.17 90))
     (property "Value" "R_Pack08" (id 1) (at 134.62 87.63 90))
-    (property "Footprint" "SamacSys_Parts:EXB2HV_1" (id 2) (at 134.62 88.265 90)
+    (property "Footprint" "footprints:EXB2HV_1" (id 2) (at 134.62 88.265 90)
       (effects (font (size 1.27 1.27)) hide)
     )
@@
     )
     (path "/4012fd8a-8fea-421b-a73e-f3dc43ce343b"
-      (reference "D1") (unit 1) (value "LED") (footprint "SamacSys_Parts:LEDC1006X25N")
+      (reference "D1") (unit 1) (value "LED") (footprint "footprints:LEDC1006X25N")
     )
     (path "/2b2281f2-5588-448e-a177-2283f74f98c6"
@@
     )
     (path "/35ee9526-dfeb-43ab-a292-2f0c25901734"
-      (reference "RN1") (unit 1) (value "R_Pack08") (footprint "SamacSys_Parts:EXB2HV_1")
+      (reference "RN1") (unit 1) (value "R_Pack08") (footprint "footprints:EXB2HV_1")
     )
     (path "/d0962256-c7ae-438a-a071-11ced85dd3a6"
-      (reference "RN2") (unit 1) (value "R_Pack08") (footprint "SamacSys_Parts:EXB2HV_1")
+      (reference "RN2") (unit 1) (value "R_Pack08") (footprint "footprints:EXB2HV_1")
     )
     (path "/c9b0f093-79f7-44a9-9a01-140d009dab54"

Commit message: Update resistors to 0805s
Parts:
- R1, R10, R11, R12, R13, R14, R15, R16, R17, R18, R19, R2, R20, R21, R22, R23, R24, R3, R4, R5, R6, R7, R8, R9: footprint Resistor_SMD:R_0402_1005Metric_Pad0.72x0.64mm_HandSolder -> Resistor_SMD:R_0805_2012Metric_Pad1.20x1.40mm_HandSolder

Commit message: Replace LED with 0805
Parts:
- D1: footprint footprints:LEDC1006X25N -> LED_SMD:LED_0805_2012Metric_Pad1.15x1.40mm_HandSolder
Changed lines of the file:
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@@
     (property "Reference" "D1" (id 0) (at 136.8425 115.57 0))
     (property "Value" "LED" (id 1) (at 136.8425 118.11 0))
-    (property "Footprint" "footprints:LEDC1006X25N" (id 2) (at 138.43 121.92 0)
+    (property "Footprint" "LED_SMD:LED_0805_2012Metric_Pad1.15x1.40mm_HandSolder" (id 2) (at 138.43 121.92 0)
       (effects (font (size 1.27 1.27)) hide)
     )
@@
     )
     (path "/4012fd8a-8fea-421b-a73e-f3dc43ce343b"
-      (reference "D1") (unit 1) (value "LED") (footprint "footprints:LEDC1006X25N")
+      (reference "D1") (unit 1) (value "LED") (footprint "LED_SMD:LED_0805_2012Metric_Pad1.15x1.40mm_HandSolder")
     )
     (path "/2b2281f2-5588-448e-a177-2283f74f98c6"

Commit message: Add mouser links to BoM
Parts:
- C1: VendorLink (none) -> https://www.mouser.com/ProductDetail/Samsung-Electro-Mechan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
- D1: VendorLink (none) -> https://www.mouser.com/ProductDetail/Wurth-Elektronik/15008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
- R1, R10, R11, R12, R13, R15, R16, R17, R18, R19, R20, R21, R22, R23, R3, R4, R5, R6, R7, R8: VendorLink (none) -> https://www.mouser.com/ProductDetail/Vishay-Dale/RCC080520K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
- R14, R2: VendorLink (none) -> https://www.mouser.com/ProductDetail/YAGEO/RC0805JR-071KL?q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
- R24: value 200 -> 33; VendorLink (none) -> https://www.mouser.com/ProductDetail/Vishay-Dale/CRCW080533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
- R9: VendorLink (none) -> https://www.mouser.com/ProductDetail/Vishay-Dale/CRCW080533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
- RN1, RN2: VendorLink (none) -> https://www.mouser.com/ProductDetail/panasonic/exb-2hv330jv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
- SW1, U1: VendorLink (none) -> https://www.mouser.com/ProductDetail/nxp/pca9548ad118/?qs=L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
